File: lora/CR2032CompactLorawanSht4x_4808/LoraTrigger.kicad_pcb (KiCad board)
At the start: 2 copper layers, 19.8 x 43.5 mm, 21 parts, among them J1 Conn_01x06, J2 Conn_02x03_Top_Bottom, J3 Conn_01x06, Q1 N-MOS, Q2 N-MOS, U1 ATmega4808-A, U3 1276Module, U4 SHT4x

Commit message: fanstelsht4x prod
Routing:
- net /SDA: track 23.3 -> 24.6 mm
- net /SS: track 14.9 -> 14.0 mm
- net /UPDI: track 30.2 -> 30.9 mm, vias 2 -> 4
- net /TXD: track 23.5 -> 23.7 mm, vias 2 -> 4
Other:
- board text added: "4808v2"
- board text added: "TX"
