File: nrf/NRFFanstelSht4x/LoraTrigger.kicad_pcb (KiCad board)
At the start: 2 copper layers, 19.8 x 30.3 mm, 12 parts, among them J1 Conn_01x04_Male, J2 Conn_01x04_Male, J3 Conn_01x02_Male, J4 Conn_01x04_Male, U1 BT, U4 SHT4x

Commit message: BT bridge fixes
Parts:
- moved R1 0.64 mm to (109.1, 66.0)
- moved R2 0.64 mm to (107.4, 66.0)
Changed lines of the file:
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@@
   )
   (footprint "halib:R_0603_Compact_hand" (layer "F.Cu")
-    (at 109.1 65.358579 90)
+    (at 109.1 66 90)
     (descr "Resistor SMD 0603, compact hand soldering")
     (tags "resistor 0603")
@@
   )
   (footprint "halib:R_0603_Compact_hand" (layer "F.Cu")
-    (at 107.4 65.358579 90)
+    (at 107.4 66 90)
     (descr "Resistor SMD 0603, compact hand soldering")
     (tags "resistor 0603")
@@
     (fp_line (start -0.3 -0.8) (end 0.3 -0.8) (layer "F.SilkS") (width 0.12))
     (fp_line (start 0.7 -0.1) (end 0.7 0.1) (layer "F.SilkS") (width 0.12))
-    (pad "1" smd rect locked (at -0.7 -0.4) (size 0.7 0.3) (layers "F.Cu" "F.Paste" "F.Mask")
+    (pad "1" smd rect (at -0.9 -0.4) (size 1.1 0.3) (layers "F.Cu" "F.Paste" "F.Mask")
       (net 8 "/SDA") (pinfunction "SDA") (pintype "bidirectional"))
-    (pad "2" smd rect (at -0.7 0.4) (size 0.7 0.3) (layers "F.Cu" "F.Paste" "F.Mask")
+    (pad "2" smd rect (at -0.9 0.4) (size 1.1 0.3) (layers "F.Cu" "F.Paste" "F.Mask")
       (net 9 "/SCL") (pinfunction "SCL") (pintype "input"))
-    (pad "3" smd rect (at 0.7 0.4) (size 0.7 0.3) (layers "F.Cu" "F.Paste" "F.Mask")
+    (pad "3" smd rect (at 0.9 0.4) (size 1.1 0.3) (layers "F.Cu" "F.Paste" "F.Mask")
       (net 6 "VCC") (pinfunction "VDD") (pintype "input"))
-    (pad "4" smd rect (at 0.7 -0.4) (size 0.7 0.3) (layers "F.Cu" "F.Paste" "F.Mask")
+    (pad "4" smd rect (at 0.9 -0.4) (size 1.1 0.3) (layers "F.Cu" "F.Paste" "F.Mask")
       (net 5 "GND") (pinfunction "GND") (pintype "input"))
   )
@@
   (segment (start 117.0993 73.09964) (end 117.173811 73.025129) (width 0.25) (layer "F.Cu") (net 7))
   (segment (start 113.8 69.459557) (end 111.570222 67.229778) (width 0.25) (layer "F.Cu") (net 8))
-  (segment (start 109.523533 65.18309) (end 108.074511 65.18309) (width 0.25) (layer "F.Cu") (net 8))
+  (segment (start 107.4 64.608579) (end 105.950489 63.159068) (width 0.25) (layer "F.Cu") (net 8))
+  (segment (start 106.4 61.8) (end 107.2 61.8) (width 0.25) (layer "F.Cu") (net 8))
+  (segment (start 108.074511 65.824511) (end 107.4 65.15) (width 0.25) (layer "F.Cu") (net 8))
+  (segment (start 105.950489 63.159068) (end 105.950489 62.249511) (width 0.25) (layer "F.Cu") (net 8))
   (segment (start 114.4 60.8) (end 114.375489 60.775489) (width 0.25) (layer "F.Cu") (net 8))
+  (segment (start 107.4 65.15) (end 107.4 64.608579) (width 0.25) (layer "F.Cu") (net 8))
   (segment (start 114.67358 79.64898) (end 113.8 78.7754) (width 0.25) (layer "F.Cu") (net 8))
-  (segment (start 107.4 64.508579) (end 107.3 64.508579) (width 0.25) (layer "F.Cu") (net 8))
-  (segment (start 107.3 64.508579) (end 106.050489 63.259068) (width 0.25) (layer "F.Cu") (net 8))
+  (segment (start 105.950489 62.249511) (end 106.4 61.8) (width 0.25) (layer "F.Cu") (net 8))
   (segment (start 111.570222 67.229778) (end 111.270222 67.229778) (width 0.25) (layer "F.Cu") (net 8))
   (segment (start 111.270222 67.229778) (end 110.8 67.7) (width 0.25) (layer "F.Cu") (net 8))
-  (segment (start 111.570222 67.229778) (end 109.523533 65.18309) (width 0.25) (layer "F.Cu") (net 8))
   (segment (start 106.850978 61.8) (end 107.3 61.8) (width 0.25) (layer "F.Cu") (net 8))
-  (segment (start 106.050489 62.149511) (end 106.3 61.9) (width 0.25) (layer "F.Cu") (net 8))
   (segment (start 114.375489 56.320489) (end 112.645 54.59) (width 0.25) (layer "F.Cu") (net 8))
   (segment (start 115.54276 79.64898) (end 114.67358 79.64898) (width 0.25) (layer "F.Cu") (net 8))
-  (segment (start 106.4 61.8) (end 107.2 61.8) (width 0.25) (layer "F.Cu") (net 8))
-  (segment (start 108.074511 65.18309) (end 107.4 64.508579) (width 0.25) (layer "F.Cu") (net 8))
+  (segment (start 110.8 67.100978) (end 109.523533 65.824511) (width 0.25) (layer "F.Cu") (net 8))
   (segment (start 112.89 54.59) (end 112.645 54.59) (width 0.25) (layer "F.Cu") (net 8))
-  (segment (start 106.050489 63.259068) (end 106.050489 62.149511) (width 0.25) (layer "F.Cu") (net 8))
   (segment (start 113.8 78.7754) (end 113.8 69.459557) (width 0.25) (layer "F.Cu") (net 8))
-  (segment (start 106.3 61.9) (end 106.4 61.8) (width 0.25) (layer "F.Cu") (net 8))
+  (segment (start 109.523533 65.824511) (end 108.074511 65.824511) (width 0.25) (layer "F.Cu") (net 8))
+  (segment (start 110.8 67.7) (end 110.8 67.100978) (width 0.25) (layer "F.Cu") (net 8))
   (segment (start 114.375489 60.775489) (end 114.375489 56.320489) (width 0.25) (layer "F.Cu") (net 8))
   (via (at 114.4 60.8) (size 0.8) (drill 0.4) (layers "F.Cu" "B.Cu") (net 8))
@@
   (segment (start 110.8 67.7) (end 114.4 64.1) (width 0.25) (layer "B.Cu") (net 8))
   (segment (start 114.4 64.1) (end 114.4 60.8) (width 0.25) (layer "B.Cu") (net 8))
-  (segment (start 106.5 62.8) (end 106.7 62.6) (width 0.25) (layer "F.Cu") (net 9))
-  (segment (start 107.991421 63.4) (end 106.9 63.4) (width 0.25) (layer "F.Cu") (net 9))
-  (segment (start 111.29571 66.00429) (end 109.8 64.508579) (width 0.25) (layer "F.Cu") (net 9))
+  (segment (start 106.4 62.9) (end 106.4 62.7) (width 0.25) (layer "F.Cu") (net 9))
+  (segment (start 114.24951 68.958089) (end 110.44142 65.15) (width 0.25) (layer "F.Cu") (net 9))
   (segment (start 115.955 57.13) (end 115.955 59.044989) (width 0.25) (layer "F.Cu") (net 9))
   (segment (start 115.955 59.044989) (end 115.099989 59.9) (width 0.25) (layer "F.Cu") (net 9))
   (segment (start 114.54346 78.54916) (end 114.249511 78.255211) (width 0.25) (layer "F.Cu") (net 9))
   (segment (start 114.249511 78.255211) (end 114.24951 68.958089) (width 0.25) (layer "F.Cu") (net 9))
-  (segment (start 106.5 63) (end 106.5 62.8) (width 0.25) (layer "F.Cu") (net 9))
-  (segment (start 109.1 64.508579) (end 107.991421 63.4) (width 0.25) (layer "F.Cu") (net 9))
-  (segment (start 106.9 63.4) (end 106.5 63) (width 0.25) (layer "F.Cu") (net 9))
-  (segment (start 114.24951 68.958089) (end 111.29571 66.00429) (width 0.25) (layer "F.Cu") (net 9))
+  (segment (start 106.4 62.7) (end 106.5 62.6) (width 0.25) (layer "F.Cu") (net 9))
+  (segment (start 109.1 65.15) (end 107.35 63.4) (width 0.25) (layer "F.Cu") (net 9))
   (segment (start 106.935704 62.6) (end 107.3 62.6) (width 0.25) (layer "F.Cu") (net 9))
+  (segment (start 106.9 63.4) (end 106.4 62.9) (width 0.25) (layer "F.Cu") (net 9))
+  (segment (start 110.44142 65.15) (end 109.1 65.15) (width 0.25) (layer "F.Cu") (net 9))
+  (segment (start 106.5 62.6) (end 107 62.6) (width 0.25) (layer "F.Cu") (net 9))
   (segment (start 106.7 62.6) (end 107.2 62.6) (width 0.25) (layer "F.Cu") (net 9))
   (segment (start 114.24951 65.55049) (end 114.3 65.5) (width 0.25) (layer "F.Cu") (net 9))
   (segment (start 115.54276 78.54916) (end 114.54346 78.54916) (width 0.25) (layer "F.Cu") (net 9))
-  (segment (start 109.8 64.508579) (end 109.1 64.508579) (width 0.25) (layer "F.Cu") (net 9))
+  (segment (start 107.35 63.4) (end 106.9 63.4) (width 0.25) (layer "F.Cu") (net 9))
   (segment (start 114.24951 68.958089) (end 114.24951 65.55049) (width 0.25) (layer "F.Cu") (net 9))
   (via (at 114.3 65.5) (size 0.8) (drill 0.4) (layers "F.Cu" "B.Cu") (net 9))
@@
     (polygon
       (pts
-        (xy 110.3 66.3)
-        (xy 106.3 66.3)
-        (xy 106.3 65.3)
-        (xy 110.3 65.3)
+        (xy 110.3 67.2)
+        (xy 106.3 67.2)
+        (xy 106.3 66.2)
+        (xy 110.3 66.2)
       )
     )

Commit message: fanstelsht4x prod
Parts:
- removed J3: Conn_01x02_Male, Connector_PinHeader_1.27mm:PinHeader_1x02_P1.27mm_Vertical
- removed J4: Conn_01x04_Male, halib:PinHeader_2x02_P1.27mm_Vertical_SMD
- added C2: 10pF, halib:C_0603_Compact_hand, F.Cu at (117.2, 80.1)
- added C3: 10pF, halib:C_0603_Compact_hand, F.Cu at (117.2, 74.5)
- added C4: C106, Capacitor_SMD:C_1206_3216Metric_Pad1.33x1.80mm_HandSolder, F.Cu at (104.2, 60.4)
- added Q1: Q_PMOS_GSD, Package_TO_SOT_SMD:SOT-23, F.Cu at (114.2, 67.4)
- added R4: 100k, halib:R_0603_Compact_hand, F.Cu at (114.2, 70.1)
- added Y1: Crystal_Small, Crystal:Crystal_SMD_MicroCrystal_CM9V-T1A-2Pin_1.6x1.0mm, F.Cu at (117.2, 77.3)
- J1: value Conn_01x04_Male -> Conn_02x04_Odd_Even; footprint Connector_PinHeader_2.54mm:PinHeader_1x04_P2.54mm_Vertical_SMD_Pin1Left -> Connector_PinSocket_2.54mm:PinSocket_2x04_P2.54mm_Vertical_SMD
- J2: value Conn_01x04_Male -> tc2030; footprint Connector_PinHeader_2.54mm:PinHeader_1x04_P2.54mm_Vertical_SMD_Pin1Left -> halib:TC2030
- U1: value BT -> BT40F
- moved J2 14.6 mm to (103.6, 68.3), turned to 180 degrees
- moved D1 11.5 mm to (101.8, 56.8), turned to 180 degrees
- moved C1 10.3 mm to (99.9, 63.4), turned to -90 degrees
- moved J1 10.0 mm to (112.5, 60.5), turned to 90 degrees
- moved R3 9.79 mm to (102.2, 58.4), turned to 180 degrees
- moved U4 5.75 mm to (102.3, 63.5), turned to 180 degrees
- moved BT1 3.21 mm to (108.2, 68.8)
- moved R1 2.50 mm to (111.1, 67.5)
- moved R2 2.50 mm to (109.4, 67.5)
- moved U1 0.93 mm to (115.2, 71.3)
Connections:
- J1 pad 1: VCC -> /SDA
- J1 pad 2: /SWDIO -> GND
- J1 pad 3: /SWDCLK -> /SCL
- J1 pad 4: GND -> VCC
- J2 pad 1: /SDA -> VCC
- J2 pad 2: /SCL -> /SWDIO
- J2 pad 3: VCC -> /RESET
- J2 pad 4: GND -> /SWDCLK
- U1 pad P$3: unconnected-(U1-PadP$3) -> /XL1
- U1 pad P$4: unconnected-(U1-PadP$4) -> /XL2
Routing:
- net /SWDIO: track 28.0 -> 13.1 mm
- net /LED: track 8.96 -> 22.3 mm, vias 0 -> 2
- net /P004: track 11.3 -> 0.00 mm
- net /V2: track 0.00 -> 8.95 mm
- net /SWDCLK: track 20.4 -> 11.5 mm
- net /P003: track 2.97 -> 10.4 mm
- net /SDA: track 41.3 -> 34.4 mm
- net /P002: track 5.02 -> 11.5 mm
- net GND: track 16.6 -> 22.8 mm, vias 5 -> 10
- net /RESET: track 6.88 -> 11.7 mm
- net /XL2: track 0.00 -> 3.18 mm
- net /XL1: track 0.00 -> 3.18 mm
- net VCC: track 20.8 -> 18.4 mm, vias 5 -> 3
- net /SWO: track 10.1 -> 7.83 mm
- net /SCL: track 35.3 -> 33.4 mm
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Other:
- board size 19.8 x 30.3 mm -> 19.8 x 27.5 mm
- board text added: "GND"
- board text added: "P2"
- board text added: "P3"
- board text added: "SCL"
- board text added: "SDA"
- board text added: "V+"
- board text added: "V2"
