File: nrf/NRFFanstelSht4x/LoraTrigger.kicad_sch (KiCad schematic)
At the start: 12 parts, among them J1 Conn_01x04_Male, J2 Conn_01x04_Male, J3 Conn_01x02_Male, J4 Conn_01x04_Male, U1 BT40F, U4 SHT4x

Commit message: fanstelsht4x prod
Parts:
- removed J1, J2: Conn_01x04_Male, Connector_PinHeader_2.54mm:PinHeader_1x04_P2.54mm_Vertical_SMD_Pin1Left, symbol Connector:Conn_01x04_Male
- removed J3: Conn_01x02_Male, Connector_PinHeader_1.27mm:PinHeader_1x02_P1.27mm_Vertical, symbol Connector:Conn_01x02_Male
- removed J4: Conn_01x04_Male, halib:PinHeader_2x02_P1.27mm_Vertical_SMD, symbol Connector:Conn_01x04_Male
- added C2, C3: 10pF, halib:C_0603_Compact_hand, symbol Device:C
- added C4: C106, Capacitor_SMD:C_1206_3216Metric_Pad1.33x1.80mm_HandSolder, symbol Device:C
- added J1: Conn_02x04_Odd_Even, Connector_PinSocket_2.54mm:PinSocket_2x04_P2.54mm_Vertical_SMD, symbol Connector_Generic:Conn_02x04_Odd_Even
- added J2: tc2030, halib:TC2030, symbol HASymbols:tc2030
- added Q1: Q_PMOS_GSD, Package_TO_SOT_SMD:SOT-23, symbol Device:Q_PMOS_GSD
- added R4: 100k, halib:R_0603_Compact_hand, symbol Device:R
- added Y1: Crystal_Small, Crystal:Crystal_SMD_MicroCrystal_CM9V-T1A-2Pin_1.6x1.0mm, symbol Device:Crystal_Small
Connections:
- net GND: now also C2.2, C3.2, C4.2, J1.2 (Pin_2), J1.7 (Pin_7), J2.5 (GND)
- net P002: now also J1.8 (Pin_8)
- net P003: now also J1.6 (Pin_6)
- net P005: now also Q1.1 (G), R4.1
- net RESET: now also J2.3 (nRESET)
- net SCL: now also J1.3 (Pin_3)
- net SDA: now also J1.1 (Pin_1)
- net SWDCLK: now also J2.4 (SWCLCK)
- net SWDIO: now also J2.2 (SWDIO)
- net SWO: now also J2.6 (SWO)
- net VCC: now also C4.1, J1.4 (Pin_4), J2.1 (VCC), Q1.3 (D), R4.2
- net P00 renamed XL1
- net XL1: now also C2.1, Y1.2
- net P01 renamed XL2
- net XL2: now also C3.1, Y1.1
- new net V2: J1.5 (Pin_5), Q1.2 (S)
