File: nrf/NrfEsp/LoraTrigger.kicad_pcb (KiCad board)
At the start: 2 copper layers, 29.2 x 50.8 mm, 2 parts, among them U1 BT40F, U2 WeMos_D1_mini

Commit message: BT bridge fixes
Parts:
- moved U2 28.0 mm to (120.0, 58.0), turned to 180 degrees
Connections:
- U2 pad 10: unconnected-(U2-Pad10) -> GND
- U2 pad 12: unconnected-(U2-Pad12) -> /SCL
- U2 pad 13: unconnected-(U2-Pad13) -> /SDA
- U2 pad 9: unconnected-(U2-Pad9) -> VCC
Routing:
- net /SCL: track 0.00 -> 39.8 mm
- net /SDA: track 0.00 -> 38.3 mm
- net GND: track 0.00 -> 1.78 mm, vias 0 -> 1

Commit message: fanstelsht4x prod
Parts:
- added J1: tc2030, halib:TC2030, F.Cu at (97.1, 71.5)
Routing:
- net /SWDCLK: track 0.00 -> 19.6 mm
- net /SWO: track 0.00 -> 13.4 mm
- net /SWDIO: track 0.00 -> 13.2 mm
- net /RESET: track 0.00 -> 10.2 mm
- net GND: track 1.78 -> 3.94 mm, vias 1 -> 2
Changed lines of the file:
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@@
   (net 27 "unconnected-(U2-Pad15)")
   (net 28 "unconnected-(U2-Pad16)")
+  (footprint "halib:TC2030" (layer "F.Cu")
+    (at 97.1 71.5 90)
+    (descr "Tag-Connect TC2030-NL footprint by carloscuev@gmail.com")
+    (tags "Tag-Connect TC2030-NL")
+    (property "Sheetfile" "LoraTrigger.kicad_sch")
+    (property "Sheetname" "")
+    (clearance 0.127)
+    (attr exclude_from_pos_files)
+    (fp_text reference "J1" (at -3.025 -2.075 90) (layer "F.SilkS") hide
+      (effects (font (size 0.4 0.4) (thickness 0.1)))
+    )
+    (fp_text value "tc2030" (at 0 2.667 90) (layer "F.SilkS") hide
+      (effects (font (size 0.75692 0.75692) (thickness 0.127)))
+    )
+    (fp_line (start -3.2639 -0.7239) (end -2.0828 -1.905) (layer "F.SilkS") (width 0.127))
+    (fp_line (start 2.6035 1.905) (end -2.0828 1.905) (layer "F.SilkS") (width 0.127))
+    (fp_line (start -3.2639 0.7239) (end -2.0828 1.905) (layer "F.SilkS") (width 0.127))
+    (fp_line (start 3.556 -0.9525) (end 3.556 0.9525) (layer "F.SilkS") (width 0.127))
+    (fp_line (start 2.6035 -1.905) (end -2.0828 -1.905) (layer "F.SilkS") (width 0.127))
+    (fp_arc (start 3.556 0.9525) (mid 3.277019 1.626019) (end 2.6035 1.905) (layer "F.SilkS") (width 0.127))
+    (fp_arc (start -3.2639 0.7239) (mid -3.563749 0) (end -3.2639 -0.7239) (layer "F.SilkS") (width 0.127))
+    (fp_arc (start 2.6035 -1.905) (mid 3.277019 -1.626019) (end 3.556 -0.9525) (layer "F.SilkS") (width 0.127))
+    (pad "" np_thru_hole circle locked (at 2.54 -1.016 90) (size 0.98552 0.98552) (drill 0.98552) (layers *.Cu *.Mask "F.SilkS"))
+    (pad "" np_thru_hole circle locked (at 2.54 1.016 90) (size 0.98552 0.98552) (drill 0.98552) (layers *.Cu *.Mask "F.SilkS"))
+    (pad "" np_thru_hole circle locked (at -2.54 0 90) (size 0.98806 0.98806) (drill 0.98806) (layers *.Cu *.Mask "F.SilkS"))
+    (pad "1" connect circle locked (at -1.27 0.635 90) (size 0.78486 0.78486) (layers "F.Cu" "F.Mask")
+      (net 6 "VCC") (pinfunction "VCC") (pintype "power_in"))
+    (pad "2" connect circle locked (at -1.27 -0.635 90) (size 0.78486 0.78486) (layers "F.Cu" "F.Mask")
+      (net 17 "/SWDIO") (pinfunction "SWDIO") (pintype "bidirectional"))
+    (pad "3" connect circle locked (at 0 0.635 90) (size 0.78486 0.78486) (layers "F.Cu" "F.Mask")
+      (net 15 "/RESET") (pinfunction "nRESET") (pintype "input"))
+    (pad "4" connect circle locked (at 0 -0.635 90) (size 0.78486 0.78486) (layers "F.Cu" "F.Mask")
+      (net 16 "/SWDCLK") (pinfunction "SWCLCK") (pintype "input"))
+    (pad "5" connect circle locked (at 1.27 0.635 90) (size 0.78486 0.78486) (layers "F.Cu" "F.Mask")
+      (net 5 "GND") (pinfunction "GND") (pintype "power_in"))
+    (pad "6" connect circle locked (at 1.27 -0.635 90) (size 0.78486 0.78486) (layers "F.Cu" "F.Mask")
+      (net 14 "/SWO") (pinfunction "SWO") (pintype "power_in"))
+  )
   (footprint "Fanstel:BT40F" (layer "F.Cu")
     (at 119.87276 69.98593 180)
@@
   (segment (start 104.11443 72.18557) (end 104.1 72.2) (width 0.25) (layer "F.Cu") (net 5))
   (segment (start 105.87482 72.18557) (end 104.11443 72.18557) (width 0.25) (layer "F.Cu") (net 5))
+  (segment (start 99.23 70.23) (end 99.7 70.7) (width 0.25) (layer "F.Cu") (net 5))
+  (segment (start 97.735 70.23) (end 99.23 70.23) (width 0.25) (layer "F.Cu") (net 5))
   (via (at 104.1 72.2) (size 0.8) (drill 0.4) (layers "F.Cu" "B.Cu") (net 5))
+  (via (at 99.7 70.7) (size 0.8) (drill 0.4) (layers "F.Cu" "B.Cu") (net 5))
   (segment (start 97.185 50.37) (end 99.3 52.485) (width 0.25) (layer "F.Cu") (net 8))
   (segment (start 99.3 52.485) (end 99.3 59) (width 0.25) (layer "F.Cu") (net 8))
@@
   (segment (start 99.749511 50.394511) (end 99.749511 58.560721) (width 0.25) (layer "F.Cu") (net 9))
   (segment (start 118.87346 77.68467) (end 119.87276 77.68467) (width 0.25) (layer "F.Cu") (net 9))
+  (segment (start 104.767732 74.38521) (end 98.475241 68.092719) (width 0.25) (layer "F.Cu") (net 14))
+  (segment (start 105.87482 74.38521) (end 104.767732 74.38521) (width 0.25) (layer "F.Cu") (net 14))
+  (segment (start 96.951281 69.743719) (end 96.465 70.23) (width 0.25) (layer "F.Cu") (net 14))
+  (segment (start 96.951281 68.898197) (end 96.951281 69.743719) (width 0.25) (layer "F.Cu") (net 14))
+  (segment (start 97.756759 68.092719) (end 96.951281 68.898197) (width 0.25) (layer "F.Cu") (net 14))
+  (segment (start 98.475241 68.092719) (end 97.756759 68.092719) (width 0.25) (layer "F.Cu") (net 14))
+  (segment (start 105.87482 76.58485) (end 102.81985 76.58485) (width 0.25) (layer "F.Cu") (net 15))
+  (segment (start 102.81985 76.58485) (end 97.735 71.5) (width 0.25) (layer "F.Cu") (net 15))
+  (segment (start 106.9 79.5) (end 100.695978 79.5) (width 0.25) (layer "F.Cu") (net 16))
+  (segment (start 106.948631 79.451369) (end 106.9 79.5) (width 0.25) (layer "F.Cu") (net 16))
+  (segment (start 95.495978 72.469022) (end 96.465 71.5) (width 0.25) (layer "F.Cu") (net 16))
+  (segment (start 106.87412 77.68467) (end 106.948631 77.759181) (width 0.25) (layer "F.Cu") (net 16))
+  (segment (start 105.87482 77.68467) (end 106.87412 77.68467) (width 0.25) (layer "F.Cu") (net 16))
+  (segment (start 106.948631 77.759181) (end 106.948631 79.451369) (width 0.25) (layer "F.Cu") (net 16))
+  (segment (start 100.695978 79.5) (end 95.495978 74.3) (width 0.25) (layer "F.Cu") (net 16))
+  (segment (start 95.495978 74.3) (end 95.495978 72.469022) (width 0.25) (layer "F.Cu") (net 16))
+  (segment (start 100.616172 78.78449) (end 96.231449 74.399767) (width 0.25) (layer "F.Cu") (net 17))
+  (segment (start 105.87482 78.78449) (end 100.616172 78.78449) (width 0.25) (layer "F.Cu") (net 17))
+  (segment (start 96.231449 74.399767) (end 96.231449 73.003551) (width 0.25) (layer "F.Cu") (net 17))
+  (segment (start 96.231449 73.003551) (end 96.465 72.77) (width 0.25) (layer "F.Cu") (net 17))
   (zone (net 6) (net_name "VCC") (layer "F.Cu") (hatch edge 0.508)
     (connect_pads (clearance 0.2))
